File: ldc_tdc_driver.kicad_pcb (KiCad board)
At the start: 4 copper layers, 41 x 27 mm, 32 parts, among them J2 Conn_01x02, J3 Conn_01x02, J6 Conn_Coaxial, J7 Conn_Coaxial, J8 Conn_Coaxial, J9 Conn_Coaxial, SW1 SW_DIP_x04, U1 74LVC2GU04, U2 74HC390D,653, U3 74HC85D,653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

Commit message: Finished layout
Parts:
- R25, R26, R27, R28, R29, R30, R31, R32, R33, R35, R36: value 2.2M -> 220k
- moved J3 2.22 mm to (150.7, 65.2), turned to 90 degrees
Routing:
- net GND: track 0.00 -> 23.4 mm, vias 0 -> 21
- net /START: track 0.00 -> 23.4 mm
- net Net-(J6-Ext): track 0.00 -> 22.8 mm
- net +3V3: track 0.00 -> 20.6 mm, vias 0 -> 5
- net /B2_STOP: track 0.00 -> 19.6 mm, vias 0 -> 2
- net /BCD1: track 0.00 -> 18.7 mm
- net /B3_STOP: track 0.00 -> 18.6 mm, vias 0 -> 2
- net /BCD3: track 0.00 -> 18.0 mm
- net /BCD0: track 0.00 -> 17.9 mm
- net Net-(J3-Pin_1): track 0.00 -> 17.9 mm
- net /B1_STOP: track 0.00 -> 16.5 mm
- net /B3_START: track 0.00 -> 16.5 mm, vias 0 -> 2
- net /B2_START: track 0.00 -> 16.4 mm, vias 0 -> 2
- net /BCD2: track 0.00 -> 16.4 mm
- net /B0_STOP: track 0.00 -> 15.7 mm
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Other:
- outline, holes or cut-outs redrawn
