File: ldc_tdc_driver.kicad_sch (KiCad schematic)
At the start: 32 parts, among them J2 Conn_01x02, J3 Conn_01x02, J6 Conn_Coaxial, J7 Conn_Coaxial, J8 Conn_Coaxial, J9 Conn_Coaxial, SW1 SW_DIP_x04, U1 74LVC2GU04, U2 74HC390D,653, U3 74HC85D,653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

Commit message: Finished layout
Parts:
- R25, R26, R27, R28, R29, R30, R31, R32, R33, R35, R36: value 2.2M -> 220k; LCSC C22938 -> C22961
Changed lines of the file:
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@@
 			)
 		)
-		(property "Value" "2.2M"
+		(property "Value" "220k"
 			(at 170.942 144.7221 0)
 			(effects
@@
 			)
 		)
-		(property "LCSC" "C22938"
+		(property "LCSC" "C22961"
 			(at 170.942 142.2979 0)
 			(effects
@@
 			)
 		)
-		(property "Value" "2.2M"
+		(property "Value" "220k"
 			(at 178.562 144.7221 0)
 			(effects
@@
 			)
 		)
-		(property "LCSC" "C22938"
+		(property "LCSC" "C22961"
 			(at 178.562 142.2979 0)
 			(effects
@@
 			)
 		)
-		(property "Value" "2.2M"
+		(property "Value" "220k"
 			(at 129.032 184.0921 0)
 			(effects
@@
 			)
 		)
-		(property "LCSC" "C22938"
+		(property "LCSC" "C22961"
 			(at 129.032 181.6679 0)
 			(effects
@@
 			)
 		)
-		(property "Value" "2.2M"
+		(property "Value" "220k"
 			(at 186.182 144.7221 0)
 			(effects
@@
 			)
 		)
-		(property "LCSC" "C22938"
+		(property "LCSC" "C22961"
 			(at 186.182 142.2979 0)
 			(effects
@@
 			)
 		)
-		(property "Value" "2.2M"
+		(property "Value" "220k"
 			(at 163.322 144.7221 0)
 			(effects
@@
 			)
 		)
-		(property "LCSC" "C22938"
+		(property "LCSC" "C22961"
 			(at 163.322 142.2979 0)
 			(effects
@@
 			)
 		)
-		(property "Value" "2.2M"
+		(property "Value" "220k"
 			(at 188.722 92.6521 0)
 			(effects
@@
 			)
 		)
-		(property "LCSC" "C22938"
+		(property "LCSC" "C22961"
 			(at 188.722 90.2279 0)
 			(effects
@@
 			)
 		)
-		(property "Value" "2.2M"
+		(property "Value" "220k"
 			(at 181.102 92.6521 0)
 			(effects
@@
 			)
 		)
-		(property "LCSC" "C22938"
+		(property "LCSC" "C22961"
 			(at 181.102 90.2279 0)
 			(effects
@@
 			)
 		)
-		(property "Value" "2.2M"
+		(property "Value" "220k"
 			(at 165.862 92.6521 0)
 			(effects
@@
 			)
 		)
-		(property "LCSC" "C22938"
+		(property "LCSC" "C22961"
 			(at 165.862 90.2279 0)
 			(effects
@@
 			)
 		)
-		(property "Value" "2.2M"
+		(property "Value" "220k"
 			(at 173.482 92.6521 0)
 			(effects
@@
 			)
 		)
-		(property "LCSC" "C22938"
+		(property "LCSC" "C22961"
 			(at 173.482 90.2279 0)
 			(effects
@@
 			)
 		)
-		(property "Value" "2.2M"
+		(property "Value" "220k"
 			(at 65.532 121.8621 0)
 			(effects
@@
 			)
 		)
-		(property "LCSC" "C22938"
+		(property "LCSC" "C22961"
 			(at 65.532 119.4379 0)
 			(effects
@@
 			)
 		)
-		(property "Value" "2.2M"
+		(property "Value" "220k"
 			(at 154.432 78.6821 0)
 			(effects
@@
 			)
 		)
-		(property "LCSC" "C22938"
+		(property "LCSC" "C22961"
 			(at 154.432 76.2579 0)
 			(effects
